File: Arduino_As_Uno.kicad_pcb (KiCad board)
At the start: 2 copper layers, 68.6 x 53.3 mm, 8 parts, among them P1 Power, P2 Analog, P3 Digital, P4 Digital, P5 CONN_1, P6 CONN_1, P7 CONN_1, P8 CONN_1

Commit message: First design sent out.
Parts:
- added C1: .1u, Capacitors_SMD:C_0805_HandSoldering, F.Cu at (157.0, 88.4)
- added C4: .1u, Capacitors_SMD:C_0805_HandSoldering, F.Cu at (141.0, 111.4)
- added C5: .1u, Capacitors_SMD:C_0805_HandSoldering, F.Cu at (141.0, 105.4)
- added C6: .1u, Capacitors_SMD:C_0805_HandSoldering, F.Cu at (156.0, 83.4)
- added J1: RJ45-TRANSFO, ga-ethernet:RJ45_TRANSFO, F.Cu at (131.0, 99.4)
- added P10: CONN_01X02, Pin_Headers:Pin_Header_Straight_1x02, F.Cu at (161.0, 79.4)
- added P9: CONN_02X03, Pin_Headers:Pin_Header_Straight_2x03, F.Cu at (174.0, 86.4)
- added R1: 1k, Resistors_SMD:R_0805_HandSoldering, F.Cu at (165.0, 88.4)
- added R10: 24, Resistors_SMD:R_2512_HandSoldering, F.Cu at (141.0, 94.4)
- added R11: 2k, Resistors_SMD:R_0805_HandSoldering, F.Cu at (144.0, 105.4)
- added R12: 2k, Resistors_SMD:R_0805_HandSoldering, F.Cu at (144.0, 111.4)
- added R13: 100, Resistors_SMD:R_2512_HandSoldering, F.Cu at (137.0, 103.4)
- added R14: 2.2k, Resistors_SMD:R_0805_HandSoldering, F.Cu at (161.0, 98.4)
- added R15: 390, Resistors_SMD:R_0805_HandSoldering, F.Cu at (117.0, 84.4)
- added R16: 390, Resistors_SMD:R_0805_HandSoldering, F.Cu at (120.0, 84.4)
- added R17: 0, Resistors_SMD:R_2512_HandSoldering, F.Cu at (129.0, 109.9)
- added R2: 2.7k, Resistors_SMD:R_0805_HandSoldering, F.Cu at (153.0, 89.4)
- added R3: 1k, Resistors_SMD:R_0805_HandSoldering, F.Cu at (150.0, 92.4)
- added R4: 1k, Resistors_SMD:R_0805_HandSoldering, F.Cu at (161.0, 92.4)
- added R5: 1.7k, Resistors_SMD:R_0805_HandSoldering, F.Cu at (159.0, 92.4)
- added R6: 1k, Resistors_SMD:R_0805_HandSoldering, F.Cu at (161.0, 96.4)
- added R7: 470, Resistors_SMD:R_0805_HandSoldering, F.Cu at (165.0, 86.4)
- added R8: 390, Resistors_SMD:R_0805_HandSoldering, F.Cu at (165.0, 84.4)
- added R9: 24, Resistors_SMD:R_2512_HandSoldering, F.Cu at (141.0, 89.4)
- added U1: MAX4413, ga-ethernet:SOT-23-8, F.Cu at (155.0, 92.4)
- added U2: ASDMB, ga-ethernet:ASDMB, F.Cu at (160.0, 84.4)
Connections:
- net +3V3 renamed Net-(P1-Pad4)
- net /0(Rx) renamed Net-(P4-Pad8)
- net /10(**/SS) renamed Net-(P3-Pad8)
- net /11(**/MOSI) renamed Net-(P3-Pad7)
- net /12(MISO) renamed Net-(P3-Pad6)
- net /13(SCK) renamed Net-(P3-Pad5)
- net /6(**) renamed Net-(P4-Pad2)
- net /8 renamed Net-(P3-Pad10)
- net /9(**) renamed Net-(P3-Pad9)
- net /A0 renamed Net-(P2-Pad1)
- net /A1 renamed Net-(P2-Pad2)
- net /A2 renamed Net-(P2-Pad3)
- net /A3 renamed Net-(P2-Pad4)
- net /AREF renamed Net-(P3-Pad3)
- net /Reset renamed Net-(P1-Pad3)
- net /Vin renamed Net-(P1-Pad8)
- P1 pad 2: /IOREF -> +1V8
- P2 pad 5: /A4(SDA) -> Net-(P2-Pad5)
- P2 pad 6: /A5(SCL) -> Net-(P2-Pad6)
- P3 pad 1: /A5(SCL) -> Net-(P3-Pad1)
- P3 pad 2: /A4(SDA) -> Net-(P3-Pad2)
- P4 pad 1: /7 -> Net-(P4-Pad1)
- P4 pad 3: /5(**) -> Net-(P10-Pad1)
- P4 pad 4: /4 -> Net-(P10-Pad2)
- P4 pad 5: /3(**) -> Net-(J1-PadGA)
- P4 pad 6: /2 -> Net-(P4-Pad6)
- P4 pad 7: /1(Tx) -> Net-(J1-PadYA)
Routing:
- net GND: track 0.00 -> 225.5 mm, vias 0 -> 30
- net Net-(J1-PadYA): track 0.00 -> 74.5 mm, vias 0 -> 1
- net Net-(J1-PadGA): track 0.00 -> 74.1 mm, vias 0 -> 1
- net GNDREF: track 0.00 -> 33.6 mm, vias 0 -> 6
- net Net-(P4-Pad1): track 0.00 -> 32.1 mm
- net Net-(J1-Pad4): track 0.00 -> 31.4 mm
- net Net-(C4-Pad2): track 0.00 -> 28.7 mm
- net Net-(P4-Pad6): track 0.00 -> 27.2 mm, vias 0 -> 2
- net +1V8: track 0.00 -> 24.7 mm, vias 0 -> 4
- net Net-(P9-Pad2): track 0.00 -> 17.9 mm, vias 0 -> 1
- net Net-(R10-Pad2): track 0.00 -> 16.0 mm
- net Net-(J1-PadYK): track 0.00 -> 14.5 mm
- net Net-(R1-Pad1): track 0.00 -> 13.6 mm
- net Net-(R2-Pad1): track 0.00 -> 9.79 mm
- net Net-(J1-Pad3): track 0.00 -> 9.60 mm
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- added copper zone on B.Cu, net +1V8
- added copper zone on F.Cu, net +1V8
- added copper zone on B.Cu, net +5V
- added copper zone on B.Cu, net GND
- added copper zone on F.Cu, net GND
- added copper zone on B.Cu, net GNDREF
- added copper zone on F.Cu, net GNDREF
